Commit message: Tried Implementing Wall Follower

File: mobile_robot/model/robot.xacro (robot description, xacro)
@@ -154,3 +154,21 @@
     <xacro:inertia_wheel/>
 </link>
+<!-- I also just created this lidar to test the wall follower -->
+<link name="lidar_link">
+  <visual>
+    <geometry>
+      <cylinder radius="0.05" length="0.05"/>
+    </geometry>
+  </visual>
+  <collision>
+    <geometry>
+      <cylinder radius="0.05" length="0.05"/>
+    </geometry>
+  </collision>
+</link>
+<joint name="lidar_joint" type="fixed">
+  <parent link="body_link"/>
+  <child link="lidar_link"/>
+  <origin xyz="0.4 0 0.2" rpy="0 0 0"/>
+  </joint>
 </robot>
